Commit message: KUKA joints are now revolute without needing to specify it

File: src/kuka_model_pkg/urdf/kuka.xacro (robot description, xacro)
@@ -12,5 +12,4 @@
     <xacro:kuka_joint
         name="joint1"
-        type="revolute"
         parent="base_link"
         child="link1"
@@ -26,5 +25,4 @@
     <xacro:kuka_joint
         name="joint2"
-        type="revolute"
         parent="link1"
         child="link2"
@@ -40,5 +38,4 @@
     <xacro:kuka_joint
         name="joint3"
-        type="revolute"
         parent="link2"
         child="link3"
@@ -54,5 +51,4 @@
     <xacro:kuka_joint
         name="joint4"
-        type="revolute"
         parent="link3"
         child="link4"
@@ -68,5 +64,4 @@
     <xacro:kuka_joint
         name="joint5"
-        type="revolute"
         parent="link4"
         child="link5"
@@ -82,5 +77,4 @@
     <xacro:kuka_joint
         name="joint6"
-        type="revolute"
         parent="link5"
         child="link6"
@@ -96,5 +90,4 @@
     <xacro:kuka_joint
         name="joint7"
-        type="revolute"
         parent="link6"
         child="wrist"

File: src/kuka_model_pkg/urdf/kuka_macro.xacro (robot description, xacro)
@@ -37,8 +37,8 @@
         </link>
     </xacro:macro>
-    <!-- Kuka robot only uses revolute joint. However, it's useful to have
-       joint type as a parameter, because exercise n6 uses a prismatic joint -->
-    <xacro:macro name="kuka_joint" params="name type parent child *origin *axis effort vel limit">
-        <joint name="${name}" type="${type}">
+    <!-- Since all KUKA joints are revolute, it's not needed to specify the
+        joint type as a parameter -->
+    <xacro:macro name="kuka_joint" params="name parent child *origin *axis effort vel limit">
+        <joint name="${name}" type="revolute">
             <parent link="${parent}" />
             <child link="${child}" />
